Commit message: Zau description fully written
Zau description written with:
    UR5 with L515 on hand (hand_camera)
    Two astra cameras on body (front_body_camera and back_body_camera)
    A T265 on body (left_body_camera)
    A VLP-16 on body (lidar3d)

File: zau_description/urdf/astra.urdf.xacro (robot description, xacro)
@@ -1,85 +1,159 @@
 <?xml version="1.0"?>
 <robot name="sensor_astra" xmlns:xacro="http://ros.org/wiki/xacro">
-  <xacro:include filename="$(find zau2_real_description)/urdf/ur.gazebo.xacro" />
-  <!-- Xacro properties -->
-  <xacro:property name="astra_cam_py" value="-0.0125" />
-  <xacro:property name="astra_depth_rel_rgb_py" value="0.0250" />
-  <xacro:property name="astra_cam_rel_rgb_py" value="-0.0125" />
-  <xacro:property name="astra_dae_display_scale" value="0.1" />
-  <!-- Parameterised in part by the values in turtlebot_properties.urdf.xacro -->
-  <xacro:macro name="sensor_astra" params="parent prefix *origin">
-    <joint name="${prefix}_joint" type="fixed">
-      <xacro:insert_block name="origin" />
-      <parent link="${parent}" />
-      <child link="${prefix}_link" />
-    </joint>
-    <link name="${prefix}_link">
-      <!-- <visual>
-        <origin xyz="-0.03 -0.06 0" rpy="${pi} 0 ${pi/2}"/>
-        <geometry>
-          <mesh filename="package://ur_e_description/meshes/sensors/astra2.dae" scale="1 1 1"/>
-        </geometry>
-      </visual> -->
-      <collision>
-        <!-- <origin xyz="0.0 0.0 0.0" rpy="0 0 0" /> -->
-        <origin xyz="-0.01 -0.06 0" rpy="0 0 0" />
-        <geometry>
-          <box size="0.0400 0.1650 0.0300" />
-        </geometry>
-      </collision>
-      <inertial>
-        <mass value="0.564" />
-        <origin xyz="0 0 0" />
-        <inertia ixx="0.003881243" ixy="0.0" ixz="0.0"
-          iyy="0.000498940" iyz="0.0"
-          izz="0.003879257" />
-      </inertial>
-    </link>
-    <!-- add to improve set initial pose on atom -->
-    <gazebo reference="${prefix}_link">
-      <selfCollide>false</selfCollide>
-    </gazebo>
-    <joint name="${prefix}_rgb_joint" type="fixed">
-      <origin xyz="0 -0.045 0" rpy="0 0 0" />
-      <parent link="${prefix}_link" />
-      <child link="${prefix}_rgb_frame" />
-    </joint>
-    <link name="${prefix}_rgb_frame" />
-    <joint name="${prefix}_rgb_optical_joint" type="fixed">
-      <origin xyz="0 0 0" rpy="${-pi/2} 0 ${-pi/2}" />
-      <parent link="${prefix}_rgb_frame" />
-      <child link="${prefix}_rgb_optical_frame" />
-    </joint>
-    <!-- add to improve set initial pose on atom -->
-    <link name="${prefix}_rgb_optical_frame">
-      <visual>
-        <origin xyz="0.0 0.0 -0.03" rpy="${pi/2} 0 0" />
-        <geometry>
-          <mesh filename="package://zau2_real_description/meshes/sensors/astra2.dae" scale="1 1 1" />
-        </geometry>
-      </visual>
-    </link>
-    <joint name="${prefix}_depth_joint" type="fixed">
-      <origin xyz="0 -0.02 0" rpy="0 0 0" />
-      <parent link="${prefix}_link" />
-      <child link="${prefix}_depth_frame" />
-    </joint>
-    <link name="${prefix}_depth_frame" />
-    <joint name="${prefix}_depth_optical_joint" type="fixed">
-      <origin xyz="0 0 0" rpy="${-pi/2} 0 ${-pi/2}" />
-      <parent link="${prefix}_depth_frame" />
-      <child link="${prefix}_depth_optical_frame" />
-    </joint>
-       <!-- add to improve set initial pose on atom -->
-       <link name="${prefix}_depth_optical_frame">
-        <!-- <visual>
-          <origin xyz="0.0 0.0 0.0" rpy="0 0 0" />
-          <geometry> -->
-            <!-- Use a slightly smaller scale than 1, so that when both models overlap its the rgb that appears.-->
-            <!-- <mesh filename="package://t2rgb_description/meshes/sensors/astra2.dae" scale="0.98 0.98 0.98" />
-          </geometry>
-        </visual> -->
-      </link>
-    <xacro:sim_3dsensor prefix="${prefix}" />
-  </xacro:macro>
+    <!-- Xacro properties -->
+    <xacro:property name="astra_cam_py" value="-0.0125"/>
+    <xacro:property name="astra_depth_rel_rgb_py" value="0.0250"/>
+    <xacro:property name="astra_cam_rel_rgb_py" value="-0.0125"/>
+    <xacro:property name="astra_dae_display_scale" value="0.1"/>
+    <!-- Parameterised in part by the values in turtlebot_properties.urdf.xacro -->
+    <xacro:macro name="sensor_astra" params="parent prefix *origin">
+        <joint name="${prefix}_joint" type="fixed">
+            <xacro:insert_block name="origin"/>
+            <parent link="${parent}"/>
+            <child link="${prefix}_link"/>
+        </joint>
+        <link name="${prefix}_link">
+            <collision>
+                <!-- <origin xyz="0.0 0.0 0.0" rpy="0 0 0" /> -->
+                <origin xyz="-0.01 -0.06 0" rpy="0 0 0"/>
+                <geometry>
+                    <box size="0.0400 0.1650 0.0300"/>
+                </geometry>
+            </collision>
+            <inertial>
+                <mass value="0.564"/>
+                <origin xyz="0 0 0"/>
+                <inertia ixx="0.003881243" ixy="0.0" ixz="0.0"
+                         iyy="0.000498940" iyz="0.0"
+                         izz="0.003879257"/>
+            </inertial>
+        </link>
+        <gazebo reference="${prefix}_link">
+            <selfCollide>false</selfCollide>
+        </gazebo>
+        <joint name="${prefix}_rgb_joint" type="fixed">
+            <origin xyz="0 -0.045 0" rpy="0 0 0"/>
+            <parent link="${prefix}_link"/>
+            <child link="${prefix}_rgb_frame"/>
+        </joint>
+        <link name="${prefix}_rgb_frame"/>
+        <joint name="${prefix}_rgb_optical_joint" type="fixed">
+            <origin xyz="0 0 0" rpy="${-pi/2} 0 ${-pi/2}"/>
+            <!--            <origin xyz="0 0 0" rpy="0 0 0"/>-->
+            <parent link="${prefix}_rgb_frame"/>
+            <child link="${prefix}_rgb_optical_frame"/>
+        </joint>
+        <link name="${prefix}_rgb_optical_frame">
+            <visual>
+                <origin xyz="0 0 0" rpy="0 0 0"/>
+                <geometry>
+                    <mesh filename="package://mmtbot_description/meshes/atom_astra_rgb/atom_astra_rgb.dae" scale="1 1 1"/>
+                </geometry>
+            </visual>
+        </link>
+        <joint name="${prefix}_depth_joint" type="fixed">
+            <origin xyz="0 -0.02 0" rpy="0 0 0"/>
+            <parent link="${prefix}_link"/>
+            <child link="${prefix}_depth_frame"/>
+        </joint>
+        <link name="${prefix}_depth_frame"/>
+        <joint name="${prefix}_depth_optical_joint" type="fixed">
+            <origin xyz="0 0 0" rpy="${-pi/2} 0 ${-pi/2}"/>
+            <parent link="${prefix}_depth_frame"/>
+            <child link="${prefix}_depth_optical_frame"/>
+        </joint>
+        <link name="${prefix}_depth_optical_frame">
+            <visual>
+                <origin xyz="0 0 0" rpy="0 0 0"/>
+                <geometry>
+                    <!-- Use a slightly smaller scale than 1, so that when both models overlap its the rgb that appears.-->
+                    <mesh filename="package://mmtbot_description/meshes/atom_astra_depth/atom_astra_depth.dae" scale="0.98 0.98 0.98"/>
+                </geometry>
+            </visual>
+        </link>
+        <gazebo reference="${prefix}_depth_frame">
+            <sensor type="depth" name="camera">
+                <always_on>true</always_on>
+                <update_rate>10.0</update_rate>
+                <camera>
+                    <horizontal_fov>${60.0*pi/180.0}</horizontal_fov>
+                    <image>
+                        <format>B8G8R8</format>
+                        <!--                      <format>RGB_INT8</format>-->
+                        <width>640</width>
+                        <height>480</height>
+                    </image>
+                    <clip>
+                        <near>0.10</near>
+                        <far>8.0</far>
+                    </clip>
+                </camera>
+                <plugin name="${prefix}_depth_camera_controller" filename="libgazebo_ros_openni_kinect.so">
+                    <cameraName>${prefix}</cameraName>
+                    <alwaysOn>true</alwaysOn>
+                    <updateRate>10.0</updateRate>
+                    <!--                                      <imageTopicName>rgb/image_raw</imageTopicName>-->
+                    <imageTopicName>null</imageTopicName>
+                    <cameraInfoTopicName>null/camera_info</cameraInfoTopicName>
+                    <depthImageTopicName>depth/image_raw</depthImageTopicName>
+                    <pointCloudTopicName>depth/points</pointCloudTopicName>
+                    <!--                  <cameraInfoTopicName>rgb/camera_info</cameraInfoTopicName>-->
+                    <depthImageCameraInfoTopicName>depth/camera_info</depthImageCameraInfoTopicName>
+                    <frameName>${prefix}_depth_optical_frame</frameName>
+                    <!--                  <frameName>${prefix}_rgb_optical_frame</frameName>-->
+                    <!--                  <frameName>${prefix}_link</frameName>-->
+                    <!-- Apparently this is not used-->
+                    <baseline>0.1</baseline>
+                    <!--                  <hackBaseline>2</hackBaseline>-->
+                    <distortion_k1>0.0</distortion_k1>
+                    <distortion_k2>0.0</distortion_k2>
+                    <distortion_k3>0.0</distortion_k3>
+                    <distortion_t1>0.0</distortion_t1>
+                    <distortion_t2>0.0</distortion_t2>
+                    <pointCloudCutoff>0.4</pointCloudCutoff>
+                </plugin>
+            </sensor>
+        </gazebo>
+        <gazebo reference="${prefix}_rgb_frame">
+            <sensor type="camera" name="camera">
+                <update_rate>30.0</update_rate>
+                <camera>
+                    <!--                    <pose>0 0 0 ${M_PI/2} ${-M_PI/2} 0</pose>-->
+                    <horizontal_fov>${60.0*pi/180.0}</horizontal_fov>
+                    <image>
+                        <format>B8G8R8</format>
+                        <!--                      <format>RGB_INT8</format>-->
+                        <width>640</width>
+                        <height>480</height>
+                    </image>
+                    <clip>
+                        <near>0.10</near>
+                        <far>8.0</far>
+                    </clip>
+                </camera>
+                <plugin name="${prefix}_rgb_camera_controller" filename="libgazebo_ros_camera.so">
+                    <cameraName>${prefix}</cameraName>
+                    <alwaysOn>true</alwaysOn>
+                    <updateRate>0</updateRate>
+                    <imageTopicName>rgb/image_raw</imageTopicName>
+                    <!--                    <depthImageTopicName>depth/image_raw</depthImageTopicName>-->
+                    <!--                    <pointCloudTopicName>depth/points</pointCloudTopicName>-->
+                    <cameraInfoTopicName>rgb/camera_info</cameraInfoTopicName>
+                    <!--                    <depthImageCameraInfoTopicName>depth/camera_info</depthImageCameraInfoTopicName>-->
+                    <!--                    <frameName>${prefix}_depth_optical_frame</frameName>-->
+                    <frameName>${prefix}_rgb_optical_frame</frameName>
+                    <!--                  <frameName>${prefix}_link</frameName>-->
+                    <!-- Apparently this is not used-->
+                    <baseline>0.1</baseline>
+                    <!--                  <hackBaseline>2</hackBaseline>-->
+                    <distortion_k1>0.0</distortion_k1>
+                    <distortion_k2>0.0</distortion_k2>
+                    <distortion_k3>0.0</distortion_k3>
+                    <distortion_t1>0.0</distortion_t1>
+                    <distortion_t2>0.0</distortion_t2>
+                    <!--                    <pointCloudCutoff>0.4</pointCloudCutoff>-->
+                </plugin>
+            </sensor>
+        </gazebo>
+    </xacro:macro>
 </robot>

File: zau_description/urdf/moving_base_odom.urdf.xacro (robot description, xacro)
@@ -2,60 +2,30 @@
 <robot xmlns:xacro="http://ros.org/wiki/xacro" name="zau2">
     <!-- properties file -->
-    <xacro:include filename="$(find zau2_real_description)/urdf/properties.xacro"/>
+    <xacro:include filename="$(find zau_description)/urdf/properties.xacro"/>
     <xacro:property name="M_PI" value="3.1415926535897931" />
     <!-- gazebo.xacro files -->
-    <xacro:include filename="$(find zau2_real_description)/urdf/moving_base_odom.gazebo.xacro"/>
+    <xacro:include filename="$(find zau_description)/urdf/moving_base_odom.gazebo.xacro"/>
     <!-- ######################## sensors ######################## -->
-    <!-- velodyne -->
-    <!-- <xacro:arg name="gpu" default="false" />
-    <xacro:property name="gpu" value="$(arg gpu)" />
-    <xacro:arg name="organize_cloud" default="false" />
-    <xacro:property name="organize_cloud" value="$(arg organize_cloud)" />
+    <!-- Includes -->
     <xacro:include filename="$(find velodyne_description)/urdf/VLP-16.urdf.xacro" />
-    <xacro:VLP-16 parent="base_link_mb" name="velodyne" topic="/velodyne_points"
-        organize_cloud="${organize_cloud}" hz="10" samples="440" gpu="${gpu}">
+    <xacro:include filename="$(find zau_description)/urdf/astra.urdf.xacro" />
+    <xacro:include filename="$(find zau_description)/urdf/t265.urdf.xacro" />
+    <!-- Velodyne -->
+    <xacro:VLP-16 parent="base_link_mb" name="lidar3d" topic="/velodyne_points" hz="10" samples="440" gpu="true">
         <origin xyz="-0.350 0.050 0.850" rpy="0 0 0" />
-    </xacro:VLP-16> -->
-    <!-- RGB camera -->
-    <xacro:include filename="$(find zau2_real_description)/urdf/astra.urdf.xacro" />
-    <xacro:sensor_astra parent="base_link_mb" prefix="camera_mb">
+    </xacro:VLP-16>
+    <!-- Astra camera -->
+    <xacro:sensor_astra parent="base_link_mb" prefix="front_body_camera">
         <origin xyz="-0.350 0.180 0.870"
             rpy="0 0 3.14" />
     </xacro:sensor_astra>
-    <!-- intel realsense camera d415 sensor -->
-    <!-- <xacro:arg name="realsense_enabled" default="$(optenv REALSENSE_ENABLED 1)" />
-    <xacro:arg name="realsense_topic" default="$(optenv REALSENSE_TOPIC realsense)" />
-    <xacro:arg name="realsense_prefix" default="$(optenv REALSENSE_PREFIX camera_realsense)" />
-    <xacro:arg name="realsense_parent" default="$(optenv REALSENSE_PARENT base_link_mb)" />
-    <xacro:arg name="realsense_xyz" default="$(optenv REALSENSE_XYZ 0.350 -0.180 0.850)" />
-    <xacro:arg name="realsense_rpy" default="$(optenv REALSENSE_RPY 0 0 0)" /> -->
-    <!-- <material name="white">
-        <color rgba="1.0 1.0 1.0 1.0" />
-    </material> -->
-    <!-- <xacro:include filename="$(find zau2_real_description)/urdf/realsense/intel_realsense.urdf.xacro" />
-    <xacro:if value="$(arg realsense_enabled)">
-        <link name="$(arg realsense_prefix)_realsense_mountpoint" />
-        <joint name="$(arg realsense_prefix)_realsense_mountpoint_joint" type="fixed">
-            <origin xyz="$(arg realsense_xyz)" rpy="$(arg realsense_rpy)" />
-            <parent link="$(arg realsense_parent)" />
-            <child link="$(arg realsense_prefix)_realsense_mountpoint" />
-        </joint>
-        <xacro:intel_realsense_mount prefix="$(arg realsense_prefix)" topic="$(arg realsense_topic)"
-            parent_link="$(arg realsense_prefix)_realsense_mountpoint" />
-    </xacro:if> -->
-    <!-- add intel realsense l515 camera -->
-    <!-- <xacro:arg name="use_nominal_extrinsics" default="false" />
-    <xacro:arg name="add_plug" default="false" />
-    <xacro:arg name="use_mesh" default="true" />
-    <xacro:include filename="$(find zau2_real_description)/urdf/realsense/_l515.urdf.xacro" />
-    <xacro:sensor_l515 parent="base_link_mb" use_nominal_extrinsics="$(arg use_nominal_extrinsics)"
-        add_plug="$(arg add_plug)" use_mesh="$(arg use_mesh)">
-        <origin xyz="0.350 0.180 0.850" rpy="0 0 0" />
-    </xacro:sensor_l515> -->
-    <!-- add intel realsense t265 -->
-    <!-- <xacro:include filename="$(find realsense_ros_gazebo)/xacro/tracker.xacro" />
-    <xacro:realsense_T265 sensor_name="camera_t265" parent_link="base_link_mb" rate="30.0">
-        <origin rpy="0 0 0" xyz="0.350 0.060 0.860" />
-    </xacro:realsense_T265> -->
+    <xacro:sensor_astra parent="base_link_mb" prefix="back_body_camera">
+        <origin xyz="0.350 0.180 0.825"
+            rpy="0 0 0" />
+    </xacro:sensor_astra>
+    <xacro:sensor_t265 parent="base_link_mb" prefix="left_body_camera">
+        <origin xyz="0.300 -0.300 0.825"
+            rpy="0 0 ${-M_PI/2}" />
+    </xacro:sensor_t265>
     <!-- ######################## the actual robot ######################## -->
     <!-- world link -->
@@ -71,5 +41,5 @@
             <origin xyz="-0.43 -0.33 0.03" rpy="1.57 0 1.57" />
             <geometry>
-                <mesh filename="package://zau2_real_description/meshes/moving_base/moving_base.STL" scale="0.001 0.001 0.001" />
+                <mesh filename="package://zau_description/meshes/moving_base/moving_base.STL" scale="0.001 0.001 0.001" />
             </geometry>
             <material name="light_black" />
@@ -106,5 +76,5 @@
             <origin xyz="0 0 -0.055" rpy="-1.57 0 0" />
             <geometry>
-                <mesh filename="package://zau2_real_description/meshes/wheels/left_tire.stl"
+                <mesh filename="package://zau_description/meshes/robot_wheels/left_tire.stl"
                     scale="0.0025 0.0025 0.0025" />
             </geometry>
@@ -133,5 +103,5 @@
             <origin xyz="0 0 0.055" rpy="1.57 0 0" />
             <geometry>
-                <mesh filename="package://zau2_real_description/meshes/wheels/left_tire.stl"
+                <mesh filename="package://zau_description/meshes/robot_wheels/left_tire.stl"
                     scale="0.0025 0.0025 0.0025" />
             </geometry>
@@ -160,5 +130,5 @@
             <origin xyz="0.027 -0.06 0" rpy="1.57 0 0" />
             <geometry>
-                <mesh filename="package://zau2_real_description/meshes/wheels/left_tire.stl"
+                <mesh filename="package://zau_description/meshes/robot_wheels/left_tire.stl"
                     scale="0.0020 0.0020 0.0020" />
             </geometry>
@@ -188,5 +158,5 @@
             <origin xyz="0.027 -0.06 0" rpy="-1.57 0 0" />
             <geometry>
-                <mesh filename="package://zau2_real_description/meshes/wheels/left_tire.stl"
+                <mesh filename="package://zau_description/meshes/robot_wheels/left_tire.stl"
                     scale="0.0020 0.0020 0.0020" />
             </geometry>
@@ -217,5 +187,5 @@
             <origin xyz="0 -0.06 0" rpy="1.57 0 0" />
             <geometry>
-                <mesh filename="package://zau2_real_description/meshes/wheels/left_tire.stl"
+                <mesh filename="package://zau_description/meshes/robot_wheels/left_tire.stl"
                     scale="0.0020 0.0020 0.0020" />
             </geometry>
@@ -245,5 +215,5 @@
             <origin xyz="0 -0.06 0" rpy="-1.57 0 0" />
             <geometry>
-                <mesh filename="package://zau2_real_description/meshes/wheels/left_tire.stl"
+                <mesh filename="package://zau_description/meshes/robot_wheels/left_tire.stl"
                     scale="0.0020 0.0020 0.0020" />
             </geometry>

File: zau_description/urdf/zau.urdf.xacro (robot description, xacro)
@@ -8,10 +8,4 @@
     <!--  args are used with $(arg arg_name), properties are used as ${property_name}-->
     <xacro:property name="M_PI" value="3.1415926535897931" />
-    <!-- Tables properties-->
-    <xacro:property name="table_height" value="0.795"/>
-    <xacro:property name="table_width" value=".9"/>
-    <xacro:property name="table_lenght" value="0.9"/>
-    <xacro:property name="table_tabletop_thickness" value="0.015"/>
-    <xacro:property name="table_leg_radius" value="0.02"/>
     <!-- Manipulator's args and propperties -->
     <xacro:arg name="joint_limit_params" default="$(find ur_description)/config/ur10e/joint_limits.yaml"/>
@@ -26,10 +20,8 @@
     <!-- Include files-->
     <!-- ####################################### -->
-    <!-- Scene objets-->
-    <xacro:include filename="$(find mmtbot_description)/urdf/properties.xacro"/>
-    <xacro:include filename="$(find mmtbot_description)/urdf/table.macro.xacro"/>
-    <xacro:include filename="$(find mmtbot_description)/urdf/tripod.macro.xacro"/>
     <!-- Sensors-->
-    <xacro:include filename="$(find mmtbot_description)/urdf/atom_astra.urdf.xacro" />
+    <xacro:include filename="$(find zau_description)/urdf/astra.urdf.xacro" />
+    <xacro:include filename="$(find zau_description)/urdf/t265.urdf.xacro"/>
+    <xacro:include filename="$(find realsense2_description)/urdf/_l515.urdf.xacro"/>
     <xacro:include filename="$(find velodyne_description)/urdf/VLP-16.urdf.xacro"/>
     <!-- Manipulator-->
@@ -38,11 +30,4 @@
     <!-- Declare links and joints -->
     <!-- ####################################### -->
-    <!-- <link name="base_footprint"/> -->
-    <!-- Place table 1 in the scene-->
-    <!-- <xacro:table_macro name="table" parent="world" width="${table_width}"
-                       lenght="${table_lenght}" height="${table_height}"
-                       tabletop_thickness="${table_tabletop_thickness}" leg_radius="${table_leg_radius}">
-        <origin xyz="-1 0 0" rpy="0 0 ${M_PI/2}" /> -->
-    <!-- </xacro:table_macro> -->
     <!-- Place AGV -->
     <xacro:include filename="$(find zau_description)/urdf/moving_base_odom.urdf.xacro" />
@@ -65,19 +50,7 @@
         <origin xyz="-0.296 -0.1688 0.826" rpy="0.0 0.0 0.0" />
     </joint>
-    <!-- Place hand camera 1 in the scene-->
-    <xacro:sensor_astra prefix="hand_camera" parent="flange">
-        <origin xyz="-0.02 0.05 0.07" rpy="0 0.0 0" />
-    </xacro:sensor_astra>
-    <!-- Place tripod in the scene-->
-    <!-- <xacro:tripod_macro name="tripod" parent="world"> -->
-        <!-- <origin xyz="1 0 0" rpy="0 0 ${2/3*M_PI}" /> -->
-    <!-- </xacro:tripod_macro> -->
-    <!-- Put 3d lidar in the scene-->
-    <!-- <xacro:VLP-16 name="lidar" parent="tripod_left_support" topic="/lidar/points"> -->
-        <!-- <origin xyz="0 0 0.001" rpy="0 0 0" /> -->
-    <!-- </xacro:VLP-16> -->
-    <!-- Put world camera on top of tripod -->
-    <!-- <xacro:sensor_astra prefix="world_camera" parent="tripod_right_support"> -->
-        <!-- <origin xyz="0.02 0.07 0.015   " rpy="0 0.0 0" /> -->
-    <!-- </xacro:sensor_astra> -->
+    <!-- Place hand camera in the scene-->
+    <xacro:sensor_l515 name="hand_camera" parent="flange">
+        <origin xyz="0.0 0.0 0.07" rpy="0 0.0 0" />
+    </xacro:sensor_l515>
 </robot>
