Commit message: topics

File: zau_description/urdf/t265.urdf.xacro (robot description, xacro)
@@ -2,5 +2,5 @@
 <robot name="sensor_t265" xmlns:xacro="http://ros.org/wiki/xacro">
     <xacro:property name="M_PI" value="3.1415926535897931" />
-    <xacro:macro name="sensor_t265" params="parent prefix *origin">
+    <xacro:macro name="sensor_t265" params="prefix *origin">
         <link name="${prefix}_link">
             <inertial>
@@ -23,4 +23,6 @@
         </link>
   </xacro:macro>
-  <xacro:sensor_t265 prefix="vo_body"/>
+  <xacro:sensor_t265 prefix="vo_body">
+    <origin xyz="0.0 0.0 0.00" rpy="0 0.0 0" />
+  </xacro:sensor_t265>
 </robot>
