Commit message: changed camera names in URDF #919

File: zau_description/urdf/moving_base_odom.urdf.xacro (robot description, xacro)
@@ -9,6 +9,6 @@
     <!-- Includes -->
     <xacro:include filename="$(find velodyne_description)/urdf/VLP-16.urdf.xacro" />
-    <xacro:include filename="$(find zau_description)/urdf/astra.urdf.xacro" />
     <xacro:include filename="$(find zau_description)/urdf/t265.urdf.xacro" />
+    <xacro:include filename="$(find zau_description)/urdf/rgb_camera.urdf.xacro" />
     <!-- Velodyne -->
     <xacro:VLP-16 parent="base_link_mb" name="lidar3d" topic="/velodyne_points" hz="10" samples="440" gpu="true">
@@ -16,16 +16,36 @@
     </xacro:VLP-16>
     <!-- Astra camera -->
-    <xacro:sensor_astra parent="base_link_mb" prefix="front_body_camera">
-        <origin xyz="-0.350 0.180 0.870"
-            rpy="0 0 3.14" />
-    </xacro:sensor_astra>
-    <xacro:sensor_astra parent="base_link_mb" prefix="back_body_camera">
-        <origin xyz="0.350 0.180 0.825"
-            rpy="0 0 0" />
-    </xacro:sensor_astra>
-    <xacro:sensor_t265 parent="base_link_mb" prefix="left_body_camera">
-        <origin xyz="0.300 -0.300 0.825"
-            rpy="0 0 ${-M_PI/2}" />
-    </xacro:sensor_t265>
+    <!-- RGB Body Front Camera -->
+    <xacro:rgb_camera parent="base_link_mb" prefix="rgb_body_front" color_gazebo="Red">
+        <origin xyz="-0.350 0.180 0.870" rpy="0 0 3.14" />
+        <color_rgb_rviz>
+            <material name="red">
+                <color rgba="0.9 0 0 1" />
+            </material>
+        </color_rgb_rviz>
+    </xacro:rgb_camera>
+    <!-- RGB Body Back Camera -->
+    <xacro:rgb_camera parent="base_link_mb" prefix="rgb_body_back" color_gazebo="Green">
+        <origin xyz="0.350 0.180 0.825" rpy="0 0 0" />
+        <color_rgb_rviz>
+            <material name="green">
+                <color rgba="0 0.9 0 1" />
+            </material>
+        </color_rgb_rviz>
+    </xacro:rgb_camera>
+    <!-- <xacro:sensor_astra parent="base_link_mb" prefix="front_body_camera"> -->
+        <!-- <origin xyz="-0.350 0.180 0.870" -->
+            <!-- rpy="0 0 3.14" /> -->
+    <!-- </xacro:sensor_astra> -->
+<!--  -->
+    <!-- <xacro:sensor_astra parent="base_link_mb" prefix="back_body_camera"> -->
+        <!-- <origin xyz="0.350 0.180 0.825" -->
+            <!-- rpy="0 0 0" /> -->
+    <!-- </xacro:sensor_astra> -->
+<!--  -->
+    <!-- <xacro:sensor_t265 parent="base_link_mb" prefix="left_body_camera"> -->
+        <!-- <origin xyz="0.300 -0.300 0.825" -->
+            <!-- rpy="0 0 ${-M_PI/2}" /> -->
+    <!-- </xacro:sensor_t265> -->
     <!-- ######################## the actual robot ######################## -->
     <!-- world link -->

File: zau_description/urdf/zau.urdf.xacro (robot description, xacro)
@@ -21,5 +21,4 @@
     <!-- ####################################### -->
     <!-- Sensors-->
-    <xacro:include filename="$(find zau_description)/urdf/astra.urdf.xacro" />
     <xacro:include filename="$(find zau_description)/urdf/t265.urdf.xacro"/>
     <xacro:include filename="$(find realsense2_description)/urdf/_l515.urdf.xacro"/>

Commit message: Adding t265 description

File: zau_description/urdf/moving_base_odom.urdf.xacro (robot description, xacro)
@@ -9,5 +9,4 @@
     <!-- Includes -->
     <xacro:include filename="$(find velodyne_description)/urdf/VLP-16.urdf.xacro" />
-    <xacro:include filename="$(find zau_description)/urdf/t265.urdf.xacro" />
     <xacro:include filename="$(find zau_description)/urdf/rgb_camera.urdf.xacro" />
     <!-- Velodyne -->
@@ -34,18 +33,4 @@
         </color_rgb_rviz>
     </xacro:rgb_camera>
-    <!-- <xacro:sensor_astra parent="base_link_mb" prefix="front_body_camera"> -->
-        <!-- <origin xyz="-0.350 0.180 0.870" -->
-            <!-- rpy="0 0 3.14" /> -->
-    <!-- </xacro:sensor_astra> -->
-<!--  -->
-    <!-- <xacro:sensor_astra parent="base_link_mb" prefix="back_body_camera"> -->
-        <!-- <origin xyz="0.350 0.180 0.825" -->
-            <!-- rpy="0 0 0" /> -->
-    <!-- </xacro:sensor_astra> -->
-<!--  -->
-    <!-- <xacro:sensor_t265 parent="base_link_mb" prefix="left_body_camera"> -->
-        <!-- <origin xyz="0.300 -0.300 0.825" -->
-            <!-- rpy="0 0 ${-M_PI/2}" /> -->
-    <!-- </xacro:sensor_t265> -->
     <!-- ######################## the actual robot ######################## -->
     <!-- world link -->

File: zau_description/urdf/t265.urdf.xacro (robot description, xacro)
@@ -3,9 +3,4 @@
     <xacro:property name="M_PI" value="3.1415926535897931" />
     <xacro:macro name="sensor_t265" params="parent prefix *origin">
-        <joint name="${prefix}_joint" type="fixed">
-            <xacro:insert_block name="origin"/>
-            <parent link="${parent}"/>
-            <child link="${prefix}_link"/>
-        </joint>
         <link name="${prefix}_link">
             <inertial>
@@ -28,3 +23,4 @@
         </link>
   </xacro:macro>
+  <xacro:sensor_t265 prefix="vo_body"/>
 </robot>

File: zau_description/urdf/zau.urdf.xacro (robot description, xacro)
@@ -21,5 +21,4 @@
     <!-- ####################################### -->
     <!-- Sensors-->
-    <xacro:include filename="$(find zau_description)/urdf/t265.urdf.xacro"/>
     <xacro:include filename="$(find realsense2_description)/urdf/_l515.urdf.xacro"/>
     <xacro:include filename="$(find velodyne_description)/urdf/VLP-16.urdf.xacro"/>

Commit message: fixed sensor positions

File: zau_description/urdf/moving_base_odom.urdf.xacro (robot description, xacro)
@@ -12,10 +12,10 @@
     <!-- Velodyne -->
     <xacro:VLP-16 parent="base_link_mb" name="lidar_body" topic="/velodyne_points" hz="10" samples="440" gpu="true">
-        <origin xyz="-0.350 0.050 0.850" rpy="0 0 0" />
+        <origin xyz="0.420 0.0 0.785" rpy="0 0 0" />
     </xacro:VLP-16>
     <!-- Astra camera -->
     <!-- RGB Body Front Camera -->
     <xacro:rgb_camera parent="base_link_mb" prefix="rgb_body_front" color_gazebo="Red">
-        <origin xyz="-0.350 0.180 0.870" rpy="0 0 3.14" />
+        <origin xyz="0.420 -0.180 0.785" rpy="0 0 0" />
         <color_rgb_rviz>
             <material name="red">
@@ -26,5 +26,5 @@
     <!-- RGB Body Back Camera -->
     <xacro:rgb_camera parent="base_link_mb" prefix="rgb_body_back" color_gazebo="Green">
-        <origin xyz="0.350 0.180 0.825" rpy="0 0 0" />
+        <origin xyz="0.420 0.180 0.785" rpy="0 0 0" />
         <color_rgb_rviz>
             <material name="green">

Commit message: adjusted rgb_right rotation

File: zau_description/urdf/moving_base_odom.urdf.xacro (robot description, xacro)
@@ -17,5 +17,5 @@
     <!-- RGB Body Right Camera -->
     <xacro:rgb_camera parent="base_link_mb" prefix="rgb_body_right" color_gazebo="Red">
-        <origin xyz="0.420 -0.180 0.785" rpy="0 0 0" />
+        <origin xyz="0.420 -0.180 0.785" rpy="0 0 -${pi/4}" />
         <color_rgb_rviz>
             <material name="red">

Commit message: Adding T265 to URDF

File: zau_description/urdf/moving_base_odom.urdf.xacro (robot description, xacro)
@@ -1,4 +1,4 @@
 <?xml version="1.0"?>
-<robot xmlns:xacro="http://ros.org/wiki/xacro" name="zau2">
+<robot xmlns:xacro="http://ros.org/wiki/xacro" name="zau">
     <!-- properties file -->
     <xacro:include filename="$(find zau_description)/urdf/properties.xacro"/>
@@ -10,4 +10,5 @@
     <xacro:include filename="$(find velodyne_description)/urdf/VLP-16.urdf.xacro" />
     <xacro:include filename="$(find zau_description)/urdf/rgb_camera.urdf.xacro" />
+    <xacro:include filename="$(find zau_description)/urdf/t265.urdf.xacro" />
     <!-- Velodyne -->
     <xacro:VLP-16 parent="base_link_mb" name="lidar_body" topic="/velodyne_points" hz="10" samples="440" gpu="true">
@@ -33,4 +34,8 @@
         </color_rgb_rviz>
     </xacro:rgb_camera>
+    <!-- T265 -->
+    <xacro:sensor_t265 parent="base_link_mb" prefix="vo_camera">
+        <origin xyz="0.470 0 0.75" rpy="0 0 0" />
+    </xacro:sensor_t265>
     <!-- ######################## the actual robot ######################## -->
     <!-- world link -->

File: zau_description/urdf/t265.urdf.xacro (robot description, xacro)
@@ -3,4 +3,9 @@
     <xacro:property name="M_PI" value="3.1415926535897931" />
     <xacro:macro name="sensor_t265" params="parent prefix *origin">
+		<joint name="${prefix}_joint" type="fixed">
+			<xacro:insert_block name="origin" />
+			<parent link="${parent}" />
+			<child link="${prefix}_link" />
+		</joint>
         <link name="${prefix}_link">
             <inertial>
@@ -23,4 +28,3 @@
         </link>
   </xacro:macro>
-  <xacro:sensor_t265 prefix="vo_body"/>
 </robot>

Commit message: lardemua/atom#934 Changing zau wheels to static

File: zau_description/urdf/moving_base_odom.urdf.xacro (robot description, xacro)
@@ -76,9 +76,8 @@
     </joint>
     <!-- wheels -->
-    <joint name="wheel_left_joint" type="continuous">
+    <joint name="wheel_left_joint" type="fixed">
         <parent link="base_link_mb" />
         <child link="wheel_left_link" />
         <origin xyz="0.0 0.325 0.074" rpy="-1.57 0 0" />
-        <axis xyz="0 0 1" />
     </joint>
     <link name="wheel_left_link">
@@ -103,9 +102,8 @@
         </inertial>
     </link>
-    <joint name="wheel_right_joint" type="continuous">
+    <joint name="wheel_right_joint" type="fixed">
         <parent link="base_link_mb" />
         <child link="wheel_right_link" />
         <origin xyz="0.0 -0.325 0.074" rpy="-1.57 0 0" />
-        <axis xyz="0 0 1" />
     </joint>
     <link name="wheel_right_link">
